Commit message: xacro: added robot_description

File: iiwa_description/urdf/iiwa.gazebo.xacro (robot description, xacro)
@@ -1,9 +1,10 @@
 <?xml version="1.0"?>
 <robot xmlns:xacro="http://www.ros.org/wiki/xacro">
-  <xacro:macro name="iiwa_gazebo" params="robot_name">
+  <xacro:macro name="iiwa_gazebo" params="robot_name robot_description">
     <!-- Load Gazebo lib and set the robot namespace -->
     <gazebo>
       <plugin name="gazebo_ros_control" filename="libgazebo_ros_control.so">
         <robotNamespace>/${robot_name}</robotNamespace>
+        <robotParam>/${robot_description}</robotParam>
       </plugin>
     </gazebo>

File: iiwa_description/urdf/iiwa14.urdf.xacro (robot description, xacro)
@@ -7,4 +7,5 @@
   <xacro:arg name="hardware_interface" default="PositionJointInterface"/>
   <xacro:arg name="robot_name" default="iiwa"/>
+  <xacro:arg name="robot_param" default="/robot_description"/>
   <xacro:arg name="origin_xyz" default="0 0 0"/>
   <xacro:arg name="origin_rpy" default="0 0 0"/>
@@ -12,5 +13,5 @@
   <link name="world"/>
   <!--iiwa-->
-  <xacro:iiwa14 hardware_interface="$(arg hardware_interface)" robot_name="$(arg robot_name)" parent="world">
+  <xacro:iiwa14 hardware_interface="$(arg hardware_interface)" robot_name="$(arg robot_name)" robot_param="$(arg robot_param)" parent="world">
     <origin xyz="$(arg origin_xyz)" rpy="$(arg origin_rpy)" />
   </xacro:iiwa14>

File: iiwa_description/urdf/iiwa14.xacro (robot description, xacro)
@@ -13,5 +13,5 @@
   <xacro:property name="max_effort" value="300"/>
   <xacro:property name="max_velocity" value="10"/>
-  <xacro:macro name="iiwa14" params="parent hardware_interface robot_name *origin">
+  <xacro:macro name="iiwa14" params="parent hardware_interface robot_name robot_param *origin">
     <!--joint between {parent} and link_0-->
     <joint name="${parent}_${robot_name}_joint" type="fixed">
@@ -300,5 +300,5 @@
     </link>
     <!--Extensions -->
-    <xacro:iiwa_gazebo robot_name="${robot_name}" />
+    <xacro:iiwa_gazebo robot_name="${robot_name}" robot_param="${robot_param}" />
     <xacro:iiwa_transmission hardware_interface="${hardware_interface}"/>
   </xacro:macro>

File: iiwa_description/urdf/iiwa7.urdf.xacro (robot description, xacro)
@@ -6,11 +6,12 @@
   <xacro:include filename="$(find iiwa_description)/urdf/iiwa7.xacro"/>
   <xacro:arg name="hardware_interface" default="PositionJointInterface"/>
-  <xacro:arg name="robot_name" default="iiwa"/>
-  <xacro:arg name="origin_xyz" default="0 0 0"/>
-  <xacro:arg name="origin_rpy" default="0 0 0"/>
+  <xacro:arg name="robot_name"  default="iiwa"/>
+  <xacro:arg name="robot_param" default="/robot_description"/>
+  <xacro:arg name="origin_xyz"  default="0 0 0"/>
+  <xacro:arg name="origin_rpy"  default="0 0 0"/>
   <!-- Fix to world just for testing -->
   <link name="world"/>
   <!--iiwa-->
-  <xacro:iiwa7 hardware_interface="$(arg hardware_interface)" robot_name="$(arg robot_name)" parent="world">
+  <xacro:iiwa7 hardware_interface="$(arg hardware_interface)" robot_name="$(arg robot_name)" robot_param="$(arg robot_param)" parent="world">
     <origin xyz="$(arg origin_xyz)" rpy="$(arg origin_rpy)" />
   </xacro:iiwa7>

File: iiwa_description/urdf/iiwa7.xacro (robot description, xacro)
@@ -13,5 +13,5 @@
   <xacro:property name="max_effort" value="300"/>
   <xacro:property name="max_velocity" value="10"/>
-  <xacro:macro name="iiwa7" params="parent hardware_interface robot_name *origin">
+  <xacro:macro name="iiwa7" params="parent hardware_interface robot_name robot_param *origin">
     <!--joint between {parent} and link_0-->
     <joint name="${parent}_${robot_name}_joint" type="fixed">
@@ -294,5 +294,5 @@
     </link>
     <!--Extensions -->
-    <xacro:iiwa_gazebo robot_name="${robot_name}" />
+    <xacro:iiwa_gazebo robot_name="${robot_name}" robot_param="${robot_param}" />
     <xacro:iiwa_transmission hardware_interface="${hardware_interface}"/>
   </xacro:macro>

Commit message: nicola: gazebo xacro fix

File: iiwa_description/urdf/iiwa.gazebo.xacro (robot description, xacro)
@@ -1,10 +1,10 @@
 <?xml version="1.0"?>
 <robot xmlns:xacro="http://www.ros.org/wiki/xacro">
-  <xacro:macro name="iiwa_gazebo" params="robot_name robot_description">
+  <xacro:macro name="iiwa_gazebo" params="robot_name robot_description_param">
     <!-- Load Gazebo lib and set the robot namespace -->
     <gazebo>
       <plugin name="gazebo_ros_control" filename="libgazebo_ros_control.so">
         <robotNamespace>/${robot_name}</robotNamespace>
-        <robotParam>/${robot_description}</robotParam>
+        <robotParam>/${robot_description_param}</robotParam>
       </plugin>
     </gazebo>

File: iiwa_description/urdf/iiwa14.xacro (robot description, xacro)
@@ -13,5 +13,5 @@
   <xacro:property name="max_effort" value="300"/>
   <xacro:property name="max_velocity" value="10"/>
-  <xacro:macro name="iiwa14" params="parent hardware_interface robot_name robot_param *origin">
+  <xacro:macro name="iiwa14" params="parent hardware_interface robot_name robot_description_param *origin">
     <!--joint between {parent} and link_0-->
     <joint name="${parent}_${robot_name}_joint" type="fixed">
@@ -300,5 +300,5 @@
     </link>
     <!--Extensions -->
-    <xacro:iiwa_gazebo robot_name="${robot_name}" robot_param="${robot_param}" />
+    <xacro:iiwa_gazebo robot_name="${robot_name}" robot_description_param="${robot_description_param}" />
     <xacro:iiwa_transmission hardware_interface="${hardware_interface}"/>
   </xacro:macro>

Commit message: nicola: xacro gazebo support fixed

File: iiwa_description/urdf/iiwa.gazebo.xacro (robot description, xacro)
@@ -5,6 +5,6 @@
     <gazebo>
       <plugin name="gazebo_ros_control" filename="libgazebo_ros_control.so">
-        <robotNamespace>/${robot_name}</robotNamespace>
-        <robotParam>/${robot_description_param}</robotParam>
+        <robotNamespace>${robot_name}</robotNamespace>
+        <robotParam>${robot_description_param}</robotParam>
       </plugin>
     </gazebo>

File: iiwa_description/urdf/iiwa14.urdf.xacro (robot description, xacro)
@@ -7,5 +7,5 @@
   <xacro:arg name="hardware_interface" default="PositionJointInterface"/>
   <xacro:arg name="robot_name" default="iiwa"/>
-  <xacro:arg name="robot_param" default="/robot_description"/>
+  <xacro:arg name="robot_description_param" default="/robot_description"/>
   <xacro:arg name="origin_xyz" default="0 0 0"/>
   <xacro:arg name="origin_rpy" default="0 0 0"/>
@@ -13,5 +13,5 @@
   <link name="world"/>
   <!--iiwa-->
-  <xacro:iiwa14 hardware_interface="$(arg hardware_interface)" robot_name="$(arg robot_name)" robot_param="$(arg robot_param)" parent="world">
+  <xacro:iiwa14 hardware_interface="$(arg hardware_interface)" robot_name="$(arg robot_name)" robot_description_param="$(arg robot_description_param)" parent="world">
     <origin xyz="$(arg origin_xyz)" rpy="$(arg origin_rpy)" />
   </xacro:iiwa14>

File: iiwa_description/urdf/iiwa7.urdf.xacro (robot description, xacro)
@@ -7,5 +7,5 @@
   <xacro:arg name="hardware_interface" default="PositionJointInterface"/>
   <xacro:arg name="robot_name"  default="iiwa"/>
-  <xacro:arg name="robot_param" default="/robot_description"/>
+  <xacro:arg name="robot_description_param" default="/robot_description"/>
   <xacro:arg name="origin_xyz"  default="0 0 0"/>
   <xacro:arg name="origin_rpy"  default="0 0 0"/>
@@ -13,5 +13,5 @@
   <link name="world"/>
   <!--iiwa-->
-  <xacro:iiwa7 hardware_interface="$(arg hardware_interface)" robot_name="$(arg robot_name)" robot_param="$(arg robot_param)" parent="world">
+  <xacro:iiwa7 hardware_interface="$(arg hardware_interface)" robot_name="$(arg robot_name)" robot_description_param="$(arg robot_description_param)" parent="world">
     <origin xyz="$(arg origin_xyz)" rpy="$(arg origin_rpy)" />
   </xacro:iiwa7>

File: iiwa_description/urdf/iiwa7.xacro (robot description, xacro)
@@ -13,5 +13,5 @@
   <xacro:property name="max_effort" value="300"/>
   <xacro:property name="max_velocity" value="10"/>
-  <xacro:macro name="iiwa7" params="parent hardware_interface robot_name robot_param *origin">
+  <xacro:macro name="iiwa7" params="parent hardware_interface robot_name robot_description_param *origin">
     <!--joint between {parent} and link_0-->
     <joint name="${parent}_${robot_name}_joint" type="fixed">
@@ -294,5 +294,5 @@
     </link>
     <!--Extensions -->
-    <xacro:iiwa_gazebo robot_name="${robot_name}" robot_param="${robot_param}" />
+    <xacro:iiwa_gazebo robot_name="${robot_name}" robot_description_param="${robot_description_param}" />
     <xacro:iiwa_transmission hardware_interface="${hardware_interface}"/>
   </xacro:macro>
